Commit message: Se agrega contenedor y se corrige el movimiento

File: niryo_one_gazebo/urdf/bin.urdf (robot description, URDF)
Before this commit: robot bin, 6 links, 5 joints
Links:
- link back: geometry collision box size=0.2 0.01 0.1; visual box size=0.2 0.01 0.1
- link bottom: geometry collision box size=0.2 0.2 0.01; visual box size=0.2 0.2 0.01
- link front: geometry collision box size=0.2 0.01 0.1; visual box size=0.2 0.01 0.1
- link left: geometry collision box size=0.01 0.2 0.1; visual box size=0.01 0.2 0.1
- link right: geometry collision box size=0.01 0.2 0.1; visual box size=0.01 0.2 0.1

File: niryo_one_gazebo/urdf/conveyor_belt.urdf (robot description, URDF)
Before this commit: robot conveyor_belt, 2 links, 1 joints
Links:
- link base_link: geometry collision box size=2 0.5 0.15; visual box size=2 0.5 0.15

File: niryo_one_gazebo/urdf/red_box.urdf (robot description, URDF)
Before this commit: robot red_box, 2 links, 1 joints
Links:
- link base_link: geometry collision box size=0.1 0.075 0.025; visual box size=0.1 0.075 0.025
